File: hardware/BuckConvertor.kicad_sch (KiCad schematic)
At the start: 20 parts, among them J1 12V, J2 GND, J3 GND, J4 5V, U1 MP2303ADN

Commit message: improve version
Parts:
- removed C10, C7, C8, C9: 22uF, Capacitor_SMD:C_0805_2012Metric, symbol Device:C
- removed C3: 10uF, Capacitor_SMD:C_0805_2012Metric, symbol Device:C
- removed J1: 12V, TestPoint:TestPoint_Pad_3.0x3.0mm, symbol Connector:Conn_01x01_Female
- removed J2, J3: GND, TestPoint:TestPoint_Pad_3.0x3.0mm, symbol Connector:Conn_01x01_Female
- removed J4: 5V, TestPoint:TestPoint_Pad_3.0x3.0mm, symbol Connector:Conn_01x01_Female
- added D1: (no value), symbol Diode:1N5822
- added J1: (no value), symbol Connector:Conn_01x02_Female
- added J2: (no value), symbol Connector:Conn_01x03_Female
Connections:
- net GND: now also D1.2 (A), J1.2 (Pin_2), J2.3 (Pin_3)
- net at C5.2, R4.1: now also L1.1, J2.1 (Pin_1); no longer C6.2, L1.2
- net at R2.1, U1.2 (IN): now also C6.2, J1.1 (Pin_1)
- net at C4.1, U1.3 (SW): now also L1.2, D1.1 (K); no longer L1.1
- no-connect marks 0 -> 1
Other:
- note added: "Voltage Out = 0.925 * ( R3 + R4 ) / R3 ex. 0.925 * ( 44.2 + 10 ) / 10 = 5.01 Voltage Output"
- moved on the sheet: C1, C2, C4, C5, L1, R1, R2, R3, R4
