File: hardware/hardware.kicad_pcb (KiCad board)
At the start: 2 copper layers, 32 x 21 mm, 15 parts, among them J2 GND 5V, J3 GND, J4 VCC, U1 MP2303ADN

Commit message: rev1 project
Parts:
- removed J2: GND 5V, Connector_PinHeader_2.54mm:PinHeader_1x03_P2.54mm_Vertical
- removed J3: GND, TestPoint:TestPoint_Pad_3.0x3.0mm
- removed J4: VCC, TestPoint:TestPoint_Pad_3.0x3.0mm
- added D2: LED, LED_SMD:LED_0805_2012Metric, F.Cu at (147.1, 79.7)
- added GND: GND, TestPoint:TestPoint_Pad_3.0x3.0mm, F.Cu at (155.5, 91.0)
- added J1: OUTPUT, Connector_PinHeader_2.54mm:PinHeader_1x03_P2.54mm_Vertical, F.Cu at (137.0, 75.9)
- added R5: 300, Resistor_SMD:R_0805_2012Metric, F.Cu at (144.4, 79.7)
- added VCC: VCC, TestPoint:TestPoint_Pad_3.0x3.0mm, F.Cu at (155.5, 86.4)
- moved C1 81.6 mm to (128.3, 84.3), turned to 90 degrees
- moved C5 76.0 mm to (140.1, 80.0)
- moved L1 75.2 mm to (145.1, 86.5), turned to -90 degrees
- moved C4 73.6 mm to (135.2, 92.5), turned to 180 degrees
- moved C2 72.6 mm to (138.2, 88.3)
- moved R3 70.4 mm to (133.4, 80.0), turned to -90 degrees
- moved U1 70.3 mm to (133.3, 86.4)
- moved D1 70.2 mm to (143.7, 92.5), turned to 180 degrees
- moved R4 69.9 mm to (128.3, 80.0), turned to -90 degrees
- moved R1 69.7 mm to (138.2, 84.4), turned to -90 degrees
- moved R2 68.7 mm to (128.3, 88.4)
- moved C6 67.3 mm to (129.7, 92.5), turned to 0 degrees
Connections:
- net Net-(J2-Pin_2) renamed 5V
Routing:
- net Net-(J5-Pin_1): track 17.8 -> 43.0 mm
- net 5V: track 35.3 -> 23.3 mm, vias 2 -> 0
- net Net-(D1-K): track 26.0 -> 16.2 mm
- net Net-(U1-SS): track 11.3 -> 3.31 mm, vias 2 -> 0
- net GND: track 15.6 -> 8.67 mm, vias 10 -> 13
- net Net-(U1-COMP): track 10.8 -> 7.09 mm
- net Net-(D2-A): track 0.00 -> 2.71 mm
- net Net-(U1-FB): track 10.9 -> 8.85 mm
- net Net-(U1-EN): track 7.90 -> 6.08 mm
- net Net-(C2-Pad1): track 3.10 -> 2.04 mm
- net Net-(U1-BS): track 9.56 -> 8.94 mm
Other:
- board size 32 x 21 mm -> 32 x 42 mm
- board text added: "NoahBEC rev1"
- board text removed: "NoahBEC rev0"

Commit message: update rev2
Parts:
- removed J1: OUTPUT, Connector_PinHeader_2.54mm:PinHeader_1x03_P2.54mm_Vertical
- added 5V: 5V OUTPUT, TestPoint:TestPoint_Pad_2.0x2.0mm, F.Cu at (143.9, 74.9)
- added GND: GND OUTPUT, TestPoint:TestPoint_Pad_2.0x2.0mm, F.Cu at (147.0, 74.9)
- U1: footprint Package_SO:SOIC-8_3.9x4.9mm_P1.27mm -> Package_SO:SOIC-8-1EP_3.9x4.9mm_P1.27mm_EP2.29x3mm
- moved GND 23.4 mm to (135.7, 103.4)
- moved VCC 22.7 mm to (140.4, 103.4)
- moved R5 5.52 mm to (149.9, 79.2)
- moved C4 4.85 mm to (140.0, 93.2)
- moved D2 4.83 mm to (151.9, 79.2)
- moved R1 3.86 mm to (142.0, 84.0)
- moved C2 3.86 mm to (142.0, 87.9)
- moved R3 3.73 mm to (136.6, 78.1)
- moved R4 3.73 mm to (131.5, 78.1)
- moved L1 3.71 mm to (148.8, 86.2)
- moved U1 3.21 mm to (136.4, 85.8)
- moved C6 2.92 mm to (132.6, 92.8)
- moved D1 2.60 mm to (146.2, 93.2)
- moved C5 2.16 mm to (142.2, 79.5)
- moved C1 1.90 mm to (130.2, 84.5)
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Routing:
- net Net-(J5-Pin_1): track 43.0 -> 31.2 mm, vias 0 -> 2
- net Net-(U1-EN): track 6.08 -> 13.0 mm
- net 5V: track 23.3 -> 30.2 mm
- net Net-(U1-COMP): track 7.09 -> 12.5 mm, vias 0 -> 2
- net GND: track 8.67 -> 13.9 mm, vias 13 -> 22
- net Net-(D1-K): track 16.2 -> 20.6 mm
- net Net-(U1-BS): track 8.94 -> 7.61 mm
- net Net-(U1-FB): track 8.85 -> 10.1 mm
- net Net-(U1-SS): track 3.31 -> 4.43 mm
- net Net-(D2-A): track 2.71 -> 2.19 mm
Other:
- outline, holes or cut-outs redrawn
- board text added: "NoahBEC rev2"
- board text added: "Voltage Out = 0.925*(R3+R4)/R3 ex. 0.925*(44.2+10)/10=5.01v"
- board text removed: "NoahBEC rev1"
- board text removed: "Voltage Out = 0.925 * ( R3 + R4 ) / R3 ex. 0.925 * ( 44.2 + 10 ) / 10 = 5.01v"
