File: hardware/hardware.kicad_sch (KiCad schematic)
At the start: 15 parts, among them J2 OUTPUT, J3 GND, J4 VCC, U1 MP2303ADN

Commit message: rev1 project
Parts:
- removed J2: OUTPUT, Connector_PinHeader_2.54mm:PinHeader_1x03_P2.54mm_Vertical, symbol Connector:Conn_01x03_Female
- removed J3: GND, TestPoint:TestPoint_Pad_3.0x3.0mm, symbol Connector:Conn_01x01_Pin
- removed J4: VCC, TestPoint:TestPoint_Pad_3.0x3.0mm, symbol Connector:Conn_01x01_Pin
- added D2: LED, LED_SMD:LED_0805_2012Metric, symbol Device:LED
- added J1: OUTPUT, Connector_PinHeader_2.54mm:PinHeader_1x03_P2.54mm_Vertical, symbol Connector:Conn_01x03_Socket
- added J5: VCC, TestPoint:TestPoint_Pad_3.0x3.0mm, symbol Connector:Conn_01x01_Socket
- added J6: GND, TestPoint:TestPoint_Pad_3.0x3.0mm, symbol Connector:Conn_01x01_Socket
- added R5: 300, Resistor_SMD:R_0805_2012Metric, symbol Device:R
Connections:
- net GND: now also D2.1 (K), J1.3 (Pin_3), J6.1 (Pin_1)
- net at C6.2, R2.1, U1.2 (IN): now also J5.1 (Pin_1)
- net 5V: now reaches C5.2, L1.1, R4.1
- net 5V: now also J1.2 (Pin_2), R5.2
- new net: D2.2 (A), R5.1

Commit message: update rev2
Parts:
- removed J1: OUTPUT, Connector_PinHeader_2.54mm:PinHeader_1x03_P2.54mm_Vertical, symbol Connector:Conn_01x03_Socket
- added J2: GND OUTPUT, TestPoint:TestPoint_Pad_2.0x2.0mm, symbol Connector:Conn_01x01_Socket
- added J3: 5V OUTPUT, TestPoint:TestPoint_Pad_2.0x2.0mm, symbol Connector:Conn_01x01_Socket
- U1: footprint Package_SO:SOIC-8_3.9x4.9mm_P1.27mm -> Package_SO:SOIC-8-1EP_3.9x4.9mm_P1.27mm_EP2.29x3mm
Connections:
- net 5V: now also J3.1 (Pin_1)
- net GND: now also J2.1 (Pin_1)
- no-connect marks 1 -> 0
Changed lines of the file:
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@@
 (kicad_sch
-	(version 20231120)
+	(version 20250114)
 	(generator "eeschema")
-	(generator_version "8.0")
+	(generator_version "9.0")
 	(paper "A4")
 	(title_block
 		(title "Noah BEC")
-		(rev "1")
+		(rev "2")
+	)
+	(text "Voltage Out = 0.925 * ( R3 + R4 ) / R3\nex. 0.925 * ( 44.2 + 10 ) / 10 = 5.01 Voltage Output"
+		(exclude_from_sim no)
+		(at 116.84 118.11 0)
+		(effects
+			(font
+				(size 1.27 1.27)
+			)
+			(justify left bottom)
+		)
 	)
 	(junction
@@
 		(color 0 0 0 0)
 	)
-	(no_connect
-		(at 160.02 67.31)
-	)
 	(wire
 		(pts
@@
 			(width 0)
 			(type default)
-		)
-	)
-	(text "Voltage Out = 0.925 * ( R3 + R4 ) / R3\nex. 0.925 * ( 44.2 + 10 ) / 10 = 5.01 Voltage Output"
-		(exclude_from_sim no)
-		(at 116.84 118.11 0)
-		(effects
-			(font
-				(size 1.27 1.27)
-			)
-			(justify left bottom)
 		)
 	)
@@
 		)
 	)
+	(global_label "GND"
+		(shape input)
+		(at 165.1 67.31 0)
+		(fields_autoplaced yes)
+		(effects
+			(font
+				(size 1.27 1.27)
+			)
+			(justify left)
+		)
+		(property "Intersheetrefs" "${INTERSHEET_REFS}"
+			(at 171.3836 67.3894 0)
+			(effects
+				(font
+					(size 1.27 1.27)
+				)
+				(justify left)
+				(hide yes)
+			)
+		)
+	)
 	(global_label "5V"
 		(shape input)
@@
 		)
 	)
-	(global_label "GND"
-		(shape input)
-		(at 165.1 67.31 0)
-		(fields_autoplaced yes)
-		(effects
-			(font
-				(size 1.27 1.27)
-			)
-			(justify left)
-		)
-		(property "Intersheetrefs" "${INTERSHEET_REFS}"
-			(at 171.3836 67.3894 0)
-			(effects
-				(font
-					(size 1.27 1.27)
-				)
-				(justify left)
-				(hide yes)
-			)
-		)
-	)
 	(symbol
 		(lib_id "Diode:1N5822")
@@
 			)
 		)
-		(property "Footprint" "Package_SO:SOIC-8_3.9x4.9mm_P1.27mm"
+		(property "Footprint" "Package_SO:SOIC-8-1EP_3.9x4.9mm_P1.27mm_EP2.29x3mm"
 			(at 137.16 86.36 0)
 			(effects
@@
 				(path "/f7ea1e9b-cb91-4723-aa0e-251bb7ff6bf6"
 					(reference "R2")
+					(unit 1)
+				)
+			)
+		)
+	)
+	(symbol
+		(lib_id "Connector:Conn_01x01_Socket")
+		(at 162.56 62.23 90)
+		(unit 1)
+		(exclude_from_sim no)
+		(in_bom yes)
+		(on_board yes)
+		(dnp no)
+		(property "Reference" "J3"
+			(at 159.258 64.008 90)
+			(effects
+				(font
+					(size 1.27 1.27)
+				)
+				(justify right)
+			)
+		)
+		(property "Value" "5V OUTPUT"
+			(at 151.892 60.96 90)
+			(effects
+				(font
+					(size 1.27 1.27)
+				)
+				(justify right)
+			)
+		)
+		(property "Footprint" "TestPoint:TestPoint_Pad_2.0x2.0mm"
+			(at 162.56 62.23 0)
+			(effects
+				(font
+					(size 1.27 1.27)
+				)
+				(hide yes)
+			)
+		)
+		(property "Datasheet" "~"
+			(at 162.56 62.23 0)
+			(effects
+				(font
+					(size 1.27 1.27)
+				)
+				(hide yes)
+			)
+		)
+		(property "Description" "Generic connector, single row, 01x01, script generated"
+			(at 162.56 62.23 0)
+			(effects
+				(font
+					(size 1.27 1.27)
+				)
+				(hide yes)
+			)
+		)
+		(pin "1"
+		)
+		(instances
+			(project ""
+				(path "/f7ea1e9b-cb91-4723-aa0e-251bb7ff6bf6"
+					(reference "J3")
 					(unit 1)
 				)
@@
 			)
 		)
+		(property "Sim.Pins" "1=K 2=A"
+			(at 147.32 52.07 0)
+			(effects
+				(font
+					(size 1.27 1.27)
+				)
+				(hide yes)
+			)
+		)
 		(pin "2"
 		)
@@
 				(path "/f7ea1e9b-cb91-4723-aa0e-251bb7ff6bf6"
 					(reference "D2")
-					(unit 1)
-				)
-			)
-		)
-	)
-	(symbol
-		(lib_id "Connector:Conn_01x03_Socket")
-		(at 162.56 62.23 90)
-		(unit 1)
-		(exclude_from_sim no)
-		(in_bom yes)
-		(on_board yes)
-		(dnp no)
-		(fields_autoplaced yes)
-		(property "Reference" "J1"
-			(at 162.56 57.15 90)
-			(effects
-				(font
-					(size 1.27 1.27)
-				)
-			)
-		)
-		(property "Value" "OUTPUT"
-			(at 162.56 59.69 90)
-			(effects
-				(font
-					(size 1.27 1.27)
-				)
-			)
-		)
-		(property "Footprint" "Connector_PinHeader_2.54mm:PinHeader_1x03_P2.54mm_Vertical"
-			(at 162.56 62.23 0)
-			(effects
-				(font
-					(size 1.27 1.27)
-				)
-				(hide yes)
-			)
-		)
-		(property "Datasheet" "~"
-			(at 162.56 62.23 0)
-			(effects
-				(font
-					(size 1.27 1.27)
-				)
-				(hide yes)
-			)
-		)
-		(property "Description" "Generic connector, single row, 01x03, script generated"
-			(at 162.56 62.23 0)
-			(effects
-				(font
-					(size 1.27 1.27)
-				)
-				(hide yes)
-			)
-		)
-		(pin "3"
-		)
-		(pin "1"
-		)
-		(pin "2"
-		)
-		(instances
-			(project "hardware"
-				(path "/f7ea1e9b-cb91-4723-aa0e-251bb7ff6bf6"
-					(reference "J1")
 					(unit 1)
 				)
@@
 				(path "/f7ea1e9b-cb91-4723-aa0e-251bb7ff6bf6"
 					(reference "R1")
+					(unit 1)
+				)
+			)
+		)
+	)
+	(symbol
+		(lib_id "Connector:Conn_01x01_Socket")
+		(at 165.1 62.23 90)
+		(unit 1)
+		(exclude_from_sim no)
+		(in_bom yes)
+		(on_board yes)
+		(dnp no)
+		(fields_autoplaced yes)
+		(property "Reference" "J2"
+			(at 166.37 61.5949 90)
+			(effects
+				(font
+					(size 1.27 1.27)
+				)
+				(justify right)
+			)
+		)
+		(property "Value" "GND OUTPUT"
+			(at 166.37 64.1349 90)
+			(effects
+				(font
+					(size 1.27 1.27)
+				)
+				(justify right)
+			)
+		)
+		(property "Footprint" "TestPoint:TestPoint_Pad_2.0x2.0mm"
+			(at 165.1 62.23 0)
+			(effects
+				(font
+					(size 1.27 1.27)
+				)
+				(hide yes)
+			)
+		)
+		(property "Datasheet" "~"
+			(at 165.1 62.23 0)
+			(effects
+				(font
+					(size 1.27 1.27)
+				)
+				(hide yes)
+			)
+		)
+		(property "Description" "Generic connector, single row, 01x01, script generated"
+			(at 165.1 62.23 0)
+			(effects
+				(font
+					(size 1.27 1.27)
+				)
+				(hide yes)
+			)
+		)
+		(pin "1"
+		)
+		(instances
+			(project ""
+				(path "/f7ea1e9b-cb91-4723-aa0e-251bb7ff6bf6"
+					(reference "J2")
 					(unit 1)
 				)
@@
 		)
 	)
+	(embedded_fonts no)
 )
